File: hardware/v3/buck.kicad_sch (KiCad schematic)
At the start: 39 parts, among them J1 Conn_01x02_Pin, J6 Conn_01x03_Pin, Q1 C3M0030090K, Q3 T2N7002AK, Q4 T2N7002AK, U10 H11L1, U12 SN74LVC2G14DBV, U13 MCP9501PT-065E/OT, U14 74AHC1G02, U16 MCP6022, U17 LM555xM, U18 MCP6561-OT, U6 MCP9501PT-065E/OT, U7 UCC5350MCQDRQ1

Commit message: idk
Parts:
- R21: value 10k -> 270R
Changed lines of the file:
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@@
 			)
 		)
-		(property "Value" "10k"
+		(property "Value" "270R"
 			(at 191.008 59.69 0)
 			(effects
